Commit message: renaming

File: src/care_description/urdf/CareBot.urdf (robot description, URDF)
Before this commit: robot CareBot, 15 links, 14 joints
Links:
- link back_left_omniwheel_caster-v2: geometry collision sphere radius=0.025; visual mesh filename=package://care_description/urdf/meshes/back_left_omniwheel_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 scale=0.001 0.001 0.001
- link back_right_omniwheel_caster-v1: geometry collision sphere radius=0.025; visual mesh filename=package://care_description/urdf/meshes/back_right_omniwheel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 scale=0.001 0.001 0.001
- link base_link-v1: geometry collision box size=0.62 1.10 0.22; visual mesh filename=package://care_description/urdf/meshes/base_link-v1.stl scale=0.001 0.001 0.001
- link front_left_omniwheel_caster-v1: geometry collision sphere radius=0.025; visual mesh filename=package://care_description/urdf/meshes/front_left_omniwheel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 scale=0.001 0.001 0.001
- link front_right_omniwheel_caster-v2: geometry collision sphere radius=0.025; visual mesh filename=package://care_description/urdf/meshes/front_right_omniwhee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 scale=0.001 0.001 0.001
- link left_drive_wheel-v1: geometry collision cylinder length=0.04 radius=0.06; visual mesh filename=package://care_description/urdf/meshes/left_drive_wheel-v1.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 scale=0.001 0.001 0.001
- link lidar_scan-v1: geometry collision cylinder length=0.04 radius=0.04; visual mesh filename=package://care_description/urdf/meshes/lidar_scan-v1.stl scale=0.001 0.001 0.001
- link right_drive_wheel-v1: geometry collision cylinder length=0.04 radius=0.06; visual mesh filename=package://care_description/urdf/meshes/right_drive_wheel-v1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 scale=0.001 0.001 0.001

Commit message: initial integration (MUST TEST WITH HARDWARE)

File: src/care_description/urdf/CareBot.urdf (robot description, URDF)
Before this commit: robot CareBot, 15 links, 14 joints
Links:
- removed link rear_center_tof
- removed link rear_left_tof
- removed link rear_right_tof
- added link left_docking_camera; collision box size=0.05 0.05 0.05; visual box size=0.05 0.05 0.05
- added link left_docking_camera_optical_frame
- added link rear_center_ultrasonic; visual cylinder length=0.02 radius=0.018
- added link rear_left_ultrasonic; visual cylinder length=0.02 radius=0.018
- added link rear_right_ultrasonic; visual cylinder length=0.02 radius=0.018
- added link right_docking_camera; collision box size=0.05 0.05 0.05; visual box size=0.05 0.05 0.05
- added link right_docking_camera_optical_frame
Joints:
- removed joint base_footprint_to_front_center_tof
- removed joint base_footprint_to_front_left_tof
- removed joint base_footprint_to_front_right_tof
- removed joint base_footprint_to_rear_center_tof
- removed joint base_footprint_to_rear_left_tof
- removed joint base_footprint_to_rear_right_tof
- added joint base_link-v1_to_front_center_tof: type fixed, parent base_link-v1, child front_center_tof, origin xyz=0.0 0.54 0.32 rpy=0.0 0.0 1.5707963267948966
- added joint base_link-v1_to_front_left_tof: type fixed, parent base_link-v1, child front_left_tof, origin xyz=-0.22 0.54 0.22 rpy=0.0 0.0 1.5707963267948966
- added joint base_link-v1_to_front_right_tof: type fixed, parent base_link-v1, child front_right_tof, origin xyz=0.22 0.54 0.22 rpy=0.0 0.0 1.5707963267948966
- added joint base_link-v1_to_left_docking_camera: type fixed, parent base_link-v1, child left_docking_camera, origin xyz=0.275 0.25 1.102 rpy=0.0 0.0 0.0
- added joint base_link-v1_to_rear_center_ultrasonic: type fixed, parent base_link-v1, child rear_center_ultrasonic, origin xyz=0.0 -0.54 0.32 rpy=0.0 0.0 -1.5707963267948966
- added joint base_link-v1_to_rear_left_ultrasonic: type fixed, parent base_link-v1, child rear_left_ultrasonic, origin xyz=-0.22 -0.54 0.22 rpy=0.0 0.0 -1.5707963267948966
- added joint base_link-v1_to_rear_right_ultrasonic: type fixed, parent base_link-v1, child rear_right_ultrasonic, origin xyz=0.22 -0.54 0.22 rpy=0.0 0.0 -1.5707963267948966
- added joint base_link-v1_to_right_docking_camera: type fixed, parent base_link-v1, child right_docking_camera, origin xyz=0.275 -0.23 1.102 rpy=0.0 0.0 0.0
- added joint left_docking_camera_to_optical_frame: type fixed, parent left_docking_camera, child left_docking_camera_optical_frame, origin xyz=0.0 0.0 0.0 rpy=-1.5707963267948966 0.0 -1.5707963267948966
- added joint right_docking_camera_to_optical_frame: type fixed, parent right_docking_camera, child right_docking_camera_optical_frame, origin xyz=0.0 0.0 0.0 rpy=-1.5707963267948966 0.0 -1.5707963267948966

Commit message: rpi to stm hardware bridge

File: src/care_description/urdf/CareBot.urdf (robot description, URDF)
Before this commit: robot CareBot, 19 links, 18 joints
Links:
- link back_left_omniwheel_caster-v2: geometry collision sphere radius=0.045; visual mesh filename=package://care_description/urdf/meshes/back_left_omniwheel_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 scale=0.001 0.001 0.001
- link back_right_omniwheel_caster-v1: geometry collision sphere radius=0.045; visual mesh filename=package://care_description/urdf/meshes/back_right_omniwheel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 scale=0.001 0.001 0.001
- link front_left_omniwheel_caster-v1: geometry collision sphere radius=0.045; visual mesh filename=package://care_description/urdf/meshes/front_left_omniwheel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 scale=0.001 0.001 0.001
- link front_right_omniwheel_caster-v2: geometry collision sphere radius=0.045; visual mesh filename=package://care_description/urdf/meshes/front_right_omniwhee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 scale=0.001 0.001 0.001
